File: averera_embedded_vertical/dnt_pcb/dnt_pcb.kicad_sch (KiCad schematic)
At the start: 54 parts, among them J10 Conn_01x01_Pin, J11 Conn_01x01_Pin, U3 STM32F103C8Tx, U5 Voltage sense, U6 LM1117S-ADJ, U7 LM1117S-ADJ

Commit message: Add updated filed from krish
Parts:
- TH2: footprint Project:Thermistor -> Library:Thermistor
- U6, U7: footprint LM1117s-ADJ:1117s_ADJ -> Library:1117s_ADJ
- Z1, Z3: footprint MM3Z3V3T1G:MM3Z3V3T1G -> Diode_SMD:D_SOD-323_HandSoldering
Changed lines of the file:
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@@
 			)
 		)
-		(property "Footprint" "LM1117s-ADJ:1117s_ADJ"
+		(property "Footprint" "Library:1117s_ADJ"
 			(at 156.21 24.13 0)
 			(effects
@@
 			)
 		)
-		(property "Footprint" "MM3Z3V3T1G:MM3Z3V3T1G"
+		(property "Footprint" "Diode_SMD:D_SOD-323_HandSoldering"
 			(at 278.5735 108.6062 0)
 			(effects
@@
 			)
 		)
-		(property "Footprint" "MM3Z3V3T1G:MM3Z3V3T1G"
+		(property "Footprint" "Diode_SMD:D_SOD-323_HandSoldering"
 			(at 201.93 30.48 0)
 			(effects
@@
 			)
 		)
-		(property "Footprint" "Project:Thermistor"
+		(property "Footprint" "Library:Thermistor"
 			(at 106.68 137.16 0)
 			(effects
@@
 		(on_board yes)
 		(dnp no)
-		(fields_autoplaced yes)
 		(property "Reference" "#PWR092"
 			(at 198.12 20.689 0)
@@
 			)
 		)
-		(property "Footprint" "LM1117s-ADJ:1117s_ADJ"
+		(property "Footprint" "Library:1117s_ADJ"
 			(at 234.95 99.06 0)
 			(effects
