File: averera_embedded_vertical/dnt_pcb/dnt_pcb.kicad_pcb (KiCad board)
At the start: 2 copper layers, 100 x 100 mm, 52 parts, among them J10 Conn_01x01_Pin, J11 Conn_01x01_Pin, J12 Conn_01x01_Pin, J13 Conn_01x01_Pin, J14 Conn_01x01_Pin, J15 Conn_01x01_Pin, U2 LM1117S-3.3, U3 STM32F103C8Tx, U5 Voltage sense

Commit message: Add updated filed from krish
Parts:
- moved UART1 136.6 mm to (174.5, 68.5), turned to 0 degrees
- moved IR1 119.4 mm to (162.0, 133.5), turned to -90 degrees
- moved CAN1 105.2 mm to (148.8, 133.5), turned to -90 degrees
- moved I2C1 89.4 mm to (133.0, 133.5), turned to -90 degrees
- moved R13 82.5 mm to (93.0, 99.5), turned to 180 degrees
- moved TH1 78.3 mm to (89.5, 81.0)
- moved C6 78.1 mm to (106.5, 96.0)
- moved C7 78.1 mm to (106.5, 82.5)
- moved TH2 77.9 mm to (89.5, 93.6)
- moved IR2 76.3 mm to (114.5, 133.5), turned to -90 degrees
- moved R12 75.4 mm to (93.5, 86.9), turned to 180 degrees
- moved C1 72.2 mm to (85.5, 86.9), turned to 180 degrees
- moved C2 71.1 mm to (85.5, 99.5), turned to 180 degrees
- moved SPI1 69.9 mm to (100.5, 133.5), turned to -90 degrees
- moved Pwm_out1 61.9 mm to (174.0, 84.3), turned to 180 degrees
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Routing:
- net +3.3V: track 0.00 -> 99.5 mm
- net GND: track 0.00 -> 91.4 mm
- net SWDIO: track 0.00 -> 61.8 mm, vias 0 -> 1
- net /uart_rx: track 0.00 -> 54.4 mm
- net SWCLK: track 0.00 -> 52.9 mm, vias 0 -> 1
- net /uart_tx: track 0.00 -> 51.6 mm
- net /pot_pwm: track 0.00 -> 49.0 mm
- net /can_tx: track 0.00 -> 48.7 mm, vias 0 -> 1
- net /throttle_pwm: track 0.00 -> 48.1 mm
- net /can_rx: track 0.00 -> 48.1 mm, vias 0 -> 1
- net Net-(IR2-Pin_2): track 0.00 -> 27.5 mm
- net /i2c_sck: track 0.00 -> 22.0 mm
- net /i2c_sda: track 0.00 -> 21.2 mm
- net /controller temp: track 0.00 -> 9.12 mm
- net Net-(C2-Pad1): track 0.00 -> 8.62 mm
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
Commit message: second commit
Parts:
- removed U2: LM1117S-3.3, LM1117s-ADJ:1117s_ADJ
- added C22: 100uF, Capacitor_SMD:C_Elec_6.3x7.7, F.Cu at (4.47, 3.58)
- added C23: 10uF, Capacitor_THT:CP_Radial_D5.0mm_P2.50mm, F.Cu at (11.6, 2.77)
- added C64: 10uF, Capacitor_THT:CP_Radial_D5.0mm_P2.50mm, F.Cu at (11.6, 9.32)
- added C65: 100uF, Capacitor_SMD:C_Elec_6.3x7.7, F.Cu at (4.47, 11.7)
- added RV2: 10k, Potentiometer_THT:Potentiometer_Runtron_RM-065_Vertical, F.Cu at (1.05, 17.9)
- added RV3: 10k, Potentiometer_THT:Potentiometer_Runtron_RM-065_Vertical, F.Cu at (9.16, 17.9)
- added U6: LM1117S-ADJ, Library:1117s_ADJ, F.Cu at (27.6, 63.0)
- added U7: LM1117S-ADJ, Library:1117s_ADJ, F.Cu at (37.0, 63.0)
- added Z1: MM3Z3V3, Diode_SMD:D_SOD-323_HandSoldering, F.Cu at (21.6, 65.2)
- added Z3: MM3Z3V3, Diode_SMD:D_SOD-323_HandSoldering, F.Cu at (21.6, 68.2)
- A1, A4, A5: footprint Project:WCS1600 -> Library:WCS1600
- TH1: footprint Project:Thermistor -> Resistor_THT:R_Radial_Power_L7.0mm_W8.0mm_Px2.40mm_Py2.30mm
- TH2: footprint Project:Thermistor -> Library:Thermistor
- moved A1 83.5 mm to (172.3, 115.2)
- moved A5 82.9 mm to (88.8, 115.2), turned to -90 degrees
- moved SPI1 68.0 mm to (168.5, 133.5)
- moved IR1 67.5 mm to (94.5, 133.5), turned to 90 degrees
- renumbered Bootloader to Bootloader1
Routing:
- net GND: track 91.4 -> 199.0 mm, vias 0 -> 1
- net +3.3V: track 99.5 -> 169.4 mm
- net Net-(A5-VOUT): track 2.00 -> 49.0 mm
- net Net-(IR1-Pin_2): track 0.00 -> 37.6 mm
- net Net-(IR2-Pin_2): track 27.5 -> 27.7 mm, vias 0 -> 1
